File: pcb/MT4BTY.kicad_pcb (KiCad board)
At the start: 2 copper layers, 90.2 x 86.4 mm, 45 parts, among them J1 CX70M-24P1, J2 Conn_01x04_Male, J3 Conn_01x04_Male, J4 Conn_01x06_Female, SW1 SW_Push, SW2 SW_Push, SW3 SW_Push, SW4 SW_Push, SW5 SW_Push, U1 ATmega32U4-AU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

Commit message: [fix]fix signal path
Routing:
- net /CPU_ROW0: track 43.3 -> 50.0 mm
- net GNDPWR: track 32.7 -> 29.7 mm, vias 31 -> 37
- net /CPU_ROW1: track 44.6 -> 47.0 mm
- net /RESET: track 85.6 -> 83.8 mm, vias 0 -> 2
- net VCC: track 65.1 -> 63.8 mm
- net /A2: track 57.9 -> 56.9 mm
- net Net-(C3-Pad1): track 39.6 -> 40.6 mm
- net /MISO: track 54.6 -> 53.8 mm
- net +5V: track 143.9 -> 143.0 mm
- net /A3: track 61.2 -> 60.5 mm
- net /SCK: track 57.2 -> 57.5 mm, vias 1 -> 3
